File: mics6814/mics6814_qwiic/_autosave-mics6814_qwiic.kicad_sch (KiCad schematic)
At the start: 26 parts, among them IC1 MiCS-6814, U1 ADS1115

Commit message: Board update
Parts:
- gave numbers to parts that had none: 1
Changed lines of the file:
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@@
   (symbol (lib_id "SparkFun-Resistors:RESISTOR1206") (at 68.58 151.13 270) (unit 1)
     (in_bom yes) (on_board yes) (fields_autoplaced)
-    (property "Reference" "R?" (id 0) (at 71.12 148.59 90)
+    (property "Reference" "R8" (id 0) (at 71.12 148.59 90)
       (effects (font (size 1.143 1.143)) (justify left))
     )
@@
     )
     (path "/c3e83e7a-dcca-4a71-85b4-e5cd4b823a7d"
-      (reference "R?") (unit 1) (value "10k") (footprint "Sparkfun-Resistors:0805")
+      (reference "R8") (unit 1) (value "10k") (footprint "Sparkfun-Resistors:0805")
     )
     (path "/0f0f7bb5-ade7-4a81-82b4-43be6a8ad05c"

Commit message: Fix minor issues and MSSOP
Parts:
- U1: value ADS1115 -> (none)
Changed lines of the file:
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@@
       (effects (font (size 1.27 1.27)) (justify left))
     )
-    (property "Value" "ADS1115" (id 1) (at 212.8394 95.25 0)
+    (property "Value" "" (id 1) (at 212.8394 95.25 0)
       (effects (font (size 1.27 1.27)) (justify left))
     )
@@
     )
     (path "/0f0f7bb5-ade7-4a81-82b4-43be6a8ad05c"
-      (reference "U1") (unit 1) (value "ADS1115") (footprint "Package_SO:TSSOP-10_3x3mm_P0.5mm")
+      (reference "U1") (unit 1) (value "ADS1115") (footprint "Package_SO:MSOP-10_3x3mm_P0.5mm")
     )
     (path "/34f2ec27-e80b-49eb-847f-cbca36bc7f20"
