File: mics6814/mics6814_qwiic/mics6814_qwiic.kicad_pcb (KiCad board)
At the start: 2 copper layers, 25.4 x 17.8 mm, 26 parts, among them J1 QWIIC_CONNECTORJS-1MM, J2 QWIIC_CONNECTORJS-1MM, Q1 MOSFET_PCH-DMG2307L, U2 74HC1G04

Commit message: Flex !
Other:
- board text added: "MICS6814 qwiic V1.0"
- board text added: "by jdexyz"
- board text removed: "MICS6814 breakout board V1.0 by jdexyz"
Changed lines of the file:
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@@
     (effects (font (size 0.5 0.5) (thickness 0.125)) (justify mirror))
+  )
+  (gr_text "by jdexyz" (at 108.712 116.332) (layer "B.SilkS")
+    (effects (font (size 1 1) (thickness 0.25)) (justify left mirror))
   )
   (gr_text "0x4a" (at 115.13 111.81) (layer "B.SilkS")
@@
     (effects (font (size 0.6096 0.6096) (thickness 0.127)) (justify mirror))
   )
-  (gr_text "MICS6814 breakout \nboard V1.0\nby jdexyz" (at 124.81 107.22) (layer "B.SilkS")
+  (gr_text "MICS6814 qwiic V1.0" (at 124.714 104.648) (layer "B.SilkS")
     (effects (font (size 1.5 1.5) (thickness 0.3)) (justify left mirror))
   )
@@
     (effects (font (size 0.6096 0.6096) (thickness 0.127)))
   )
+  (gr_text "by jdexyz" (at 108.712 116.332) (layer "B.Mask")
+    (effects (font (size 1 1) (thickness 0.2)) (justify left mirror))
+  )
   (segment (start 103.52714 105.2537) (end 103.55 105.23084) (width 0.25) (layer "F.Cu") (net 1))
